File: Case top+bottom.kicad_pcb (KiCad board)
At the start: 2 copper layers, 100 x 71.1 mm, 11 parts

Commit message: Updated Case Gerbers
Parts:
- moved G*** 3.00 mm to (140.0, 88.4)
Other:
- outline, holes or cut-outs redrawn
Changed lines of the file:
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@@
   (general
     (thickness 1.6)
-    (drawings 24)
+    (drawings 26)
     (tracks 0)
     (zones 0)
@@
   )
   (module PSX_BREAKOUT:PSX_LOGO (layer F.Cu)
-    (at 139.954 91.44)
+    (at 139.954 88.44)
     (fp_text reference G*** (at 0 0) (layer F.SilkS) hide
       (effects (font (size 1.524 1.524) (thickness 0.3)))
@@
     (pad 1 np_thru_hole circle (at 0 0) (size 3.2 3.2) (drill 3.2) (layers *.Cu *.Mask))
   )
+  (gr_line (start 147.9735 99.26) (end 147.9735 111.76) (layer Edge.Cuts) (width 0.05))
+  (gr_line (start 189.954 99.26) (end 147.9735 99.26) (layer Edge.Cuts) (width 0.05))
   (gr_line (start 132.461 40.64) (end 107.95 40.64) (layer Edge.Cuts) (width 0.05))
   (gr_line (start 132.461 40.64) (end 165.735 40.64) (layer Edge.Cuts) (width 0.05))
@@
     (effects (font (size 2 2) (thickness 0.15)) (justify mirror))
   )
-  (gr_text "PSX Breakout 1.0\nTinkerplunk.com" (at 139.192 106.807) (layer F.SilkS)
+  (gr_text "PSX Breakout 1.0\nTinkerplunk.com" (at 118.96375 106.807) (layer F.SilkS)
     (effects (font (size 3 3) (thickness 0.15)))
   )
@@
   (gr_line (start 89.954 76.2) (end 89.954 111.76) (layer Edge.Cuts) (width 0.05))
   (gr_line (start 107.95 76.2) (end 89.954 76.2) (layer Edge.Cuts) (width 0.05))
-  (gr_line (start 189.954 76.2) (end 189.954 111.76) (layer Edge.Cuts) (width 0.05))
+  (gr_line (start 189.954 76.2) (end 189.954 99.26) (layer Edge.Cuts) (width 0.05))
   (gr_line (start 165.735 76.2) (end 189.954 76.2) (layer Edge.Cuts) (width 0.05))
-  (gr_line (start 189.954 111.76) (end 89.954 111.76) (layer Edge.Cuts) (width 0.05))
+  (gr_line (start 147.9735 111.76) (end 89.954 111.76) (layer Edge.Cuts) (width 0.05))
   (gr_line (start 132.461 76.2) (end 165.735 76.2) (layer Edge.Cuts) (width 0.05))
   (gr_line (start 132.461 76.2) (end 107.95 76.2) (layer Edge.Cuts) (width 0.05))
