File: PSX Breakout.sch (KiCad schematic (older format))
At the start: 24 parts, among them J1 Conn_01x12_Male, J2 Mini-DIN-4, J3 AudioJack3, J4 DB15_Female_HighDensity, J5 3x2_RCA, SW1 SW_SPDT, SW2 SW_SP3T, SW3 SW_SP3T, U1 LM1881

Commit message: Updated to 1.2
Removed sync stripper, shrunk board, added switch to select sync source of HD15 port only.
Parts:
- removed C1, C6, C8: 100nF, Capacitor_SMD:C_0603_1608Metric_Pad1.05x0.95mm_HandSolder, symbol Device:C_Small
- removed C5: 10uF, Capacitor_SMD:CP_Elec_4x5.4, symbol Device:CP1_Small
- removed C7: 10nF, Capacitor_SMD:C_0603_1608Metric_Pad1.05x0.95mm_HandSolder, symbol Device:C_Small
- removed FB1: 220R, Inductor_SMD:L_0603_1608Metric_Pad1.05x0.95mm_HandSolder, symbol Device:Ferrite_Bead_Small
- removed JP1: Jumper_3_Open, Connector_PinHeader_2.54mm:PinHeader_1x03_P2.54mm_Vertical, symbol Jumper:Jumper_3_Open
- removed R1: 470, Resistor_SMD:R_0603_1608Metric_Pad1.05x0.95mm_HandSolder, symbol Device:R_Small_US
- removed R2: 680K, Resistor_SMD:R_0603_1608Metric_Pad1.05x0.95mm_HandSolder, symbol Device:R_Small_US
- removed SW2, SW3: SW_SP3T, PSX_BREAKOUT:C&K_SP3T, symbol Switch:SW_SP3T
- removed U1: LM1881, Package_SO:SOIC-8_3.9x4.9mm_P1.27mm, symbol SCART_to_DVI-A_Compact-eagle-import:LM1881
- J3: footprint PSX_BREAKOUT:Headphone_Jack_2.5mm_SJ1-3523N -> Tinkerplunk:CUI_SJ1-3533NG
- J4: footprint Connector_Dsub:DSUB-15-HD_Female_Horizontal_P2.29x1.98mm_EdgePinOffset3.03mm_Housed_MountingHolesOffset4.94mm -> Tinkerplunk:VGA
- J5: symbol 3x2_rca:3x2_RCA -> PSX-Breakout-rescue:3x2_RCA-3x2_rca
- SW1: footprint PSX_BREAKOUT:C&K_SPDT -> Tinkerplunk:C&K_SPDT
Connections:
- net RCA_SYNC_OUT is gone; now on net CVBS: J5.1 (INSYN)
- net VGA_SYNC_OUT: now also SW1.2 (B)
- no-connect marks 9 -> 6
Changed lines of the file:
@@
-$EndComp
-$Comp
-L Switch:SW_SP3T SW3
-U 1 1 5CF73086
-P 6750 2550
-F 0 "SW3" H 6750 2225 50  0000 C CNN
-F 1 "SW_SP3T" H 6750 2316 50  0000 C CNN
-F 2 "PSX_BREAKOUT:C&K_SP3T" H 6125 2725 50  0001 C CNN
-F 3 "~" H 6125 2725 50  0001 C CNN
-	1    6750 2550
-	-1   0    0    1
-$EndComp
-$Comp
-L Switch:SW_SP3T SW2
-U 1 1 5CF757DC
-P 6700 4450
-F 0 "SW2" H 6700 4125 50  0000 C CNN
-F 1 "SW_SP3T" H 6700 4216 50  0000 C CNN
-F 2 "PSX_BREAKOUT:C&K_SP3T" H 6075 4625 50  0001 C CNN
-F 3 "~" H 6075 4625 50  0001 C CNN
-	1    6700 4450
-	-1   0    0    1
-$EndComp
-$Comp
-L Switch:SW_SPDT SW1
-U 1 1 5CF75EF3
-P 3900 3350
-F 0 "SW1" H 3900 3025 50  0000 C CNN
-F 1 "SW_SPDT" H 3900 3116 50  0000 C CNN
-F 2 "PSX_BREAKOUT:C&K_SPDT" H 3900 3350 50  0001 C CNN
-F 3 "~" H 3900 3350 50  0001 C CNN
-	1    3900 3350
-	-1   0    0    1
-$EndComp
-$Comp
-L SCART_to_DVI-A_Compact-eagle-import:LM1881 U1
-U 1 1 5CF76786
-P 5450 3600
-F 0 "U1" H 5450 4286 59  0000 C CNN
-F 1 "LM1881" H 5450 4181 59  0000 C CNN
-F 2 "Package_SO:SOIC-8_3.9x4.9mm_P1.27mm" H 5450 3600 50  0001 C CNN
-F 3 "" H 5450 3600 50  0001 C CNN
-	1    5450 3600
-	1    0    0    -1
 $EndComp
 $Comp
@@
 F 0 "J4" H 8550 3517 50  0000 C CNN
 F 1 "DB15_Female_HighDensity" H 8550 3426 50  0000 C CNN
-F 2 "Connector_Dsub:DSUB-15-HD_Female_Horizontal_P2.29x1.98mm_EdgePinOffset3.03mm_Housed_MountingHolesOffset4.94mm" H 7600 3050 50  0001 C CNN
+F 2 "Tinkerplunk:VGA" H 7600 3050 50  0001 C CNN
 F 3 " ~" H 7600 3050 50  0001 C CNN
 	1    8550 2650
@@
 $EndComp
 $Comp
-L 3x2_rca:3x2_RCA J5
+L PSX-Breakout-rescue:3x2_RCA-3x2_rca J5
 U 1 1 5CF784EC
 P 8550 5150
@@
 	1    8550 5150
 	0    1    1    0
-$EndComp
-$Comp
-L Device:C_Small C1
-U 1 1 5CF72DB5
-P 4250 3650
-F 0 "C1" V 4021 3650 50  0000 C CNN
-F 1 "100nF" V 4112 3650 50  0000 C CNN
-F 2 "Capacitor_SMD:C_0603_1608Metric_Pad1.05x0.95mm_HandSolder" H 4250 3650 50  0001 C CNN
-F 3 "~" H 4250 3650 50  0001 C CNN
-	1    4250 3650
-	0    1    1    0
-$EndComp
-$Comp
-L Device:C_Small C8
-U 1 1 5CF73331
-P 7000 3800
-F 0 "C8" H 7092 3846 50  0000 L CNN
-F 1 "100nF" H 7092 3755 50  0000 L CNN
-F 2 "Capacitor_SMD:C_0603_1608Metric_Pad1.05x0.95mm_HandSolder" H 7000 3800 50  0001 C CNN
-F 3 "~" H 7000 3800 50  0001 C CNN
-	1    7000 3800
-	1    0    0    -1
-$EndComp
-$Comp
-L Device:C_Small C6
-U 1 1 5CF73801
-P 6700 3000
-F 0 "C6" H 6792 3046 50  0000 L CNN
-F 1 "100nF" H 6792 2955 50  0000 L CNN
-F 2 "Capacitor_SMD:C_0603_1608Metric_Pad1.05x0.95mm_HandSolder" H 6700 3000 50  0001 C CNN
-F 3 "~" H 6700 3000 50  0001 C CNN
-	1    6700 3000
-	1    0    0    -1
-$EndComp
-$Comp
-L Device:C_Small C7
-U 1 1 5CF73BC9
-P 7000 3000
-F 0 "C7" H 7092 3046 50  0000 L CNN
-F 1 "10nF" H 7092 2955 50  0000 L CNN
-F 2 "Capacitor_SMD:C_0603_1608Metric_Pad1.05x0.95mm_HandSolder" H 7000 3000 50  0001 C CNN
-F 3 "~" H 7000 3000 50  0001 C CNN
-	1    7000 3000
-	1    0    0    -1
-$EndComp
-$Comp
-L Device:CP1_Small C5
-U 1 1 5CF74126
-P 6400 3000
-F 0 "C5" H 6309 2954 50  0000 R CNN
-F 1 "10uF" H 6309 3045 50  0000 R CNN
-F 2 "Capacitor_SMD:CP_Elec_4x5.4" H 6400 3000 50  0001 C CNN
-F 3 "~" H 6400 3000 50  0001 C CNN
-	1    6400 3000
-	-1   0    0    1
-$EndComp
-$Comp
-L Device:Ferrite_Bead_Small FB1
-U 1 1 5CF744BA
-P 5350 2550
-F 0 "FB1" V 5113 2550 50  0000 C CNN
-F 1 "220R" V 5204 2550 50  0000 C CNN
-F 2 "Inductor_SMD:L_0603_1608Metric_Pad1.05x0.95mm_HandSolder" V 5280 2550 50  0001 C CNN
-F 3 "~" H 5350 2550 50  0001 C CNN
-	1    5350 2550
-	0    1    1    0
-$EndComp
-$Comp
-L Device:R_Small_US R2
-U 1 1 5CF74BB3
-P 6700 3800
-F 0 "R2" H 6768 3846 50  0000 L CNN
-F 1 "680K" H 6768 3755 50  0000 L CNN
-F 2 "Resistor_SMD:R_0603_1608Metric_Pad1.05x0.95mm_HandSolder" H 6700 3800 50  0001 C CNN
-F 3 "~" H 6700 3800 50  0001 C CNN
-	1    6700 3800
-	1    0    0    -1
 $EndComp
 $Comp
@@
 BLUE_OUT
 Text GLabel 8450 4750 0    50   Input ~ 0
-RCA_SYNC_OUT
+CVBS
 Text GLabel 8250 5150 0    50   Input ~ 0
 GND
@@
 F 0 "J3" H 8270 1433 50  0000 R CNN
 F 1 "AudioJack3" H 8270 1524 50  0000 R CNN
-F 2 "PSX_BREAKOUT:Headphone_Jack_2.5mm_SJ1-3523N" H 8550 1500 50  0001 C CNN
+F 2 "Tinkerplunk:CUI_SJ1-3533NG" H 8550 1500 50  0001 C CNN
 F 3 "~" H 8550 1500 50  0001 C CNN
 	1    8550 1500
@@
 Text GLabel 8350 1600 0    50   Input ~ 0
 GND
-Text GLabel 4650 3900 0    50   Input ~ 0
-GND
-Wire Wire Line
-	6250 3300 6250 2550
-Wire Wire Line
-	6250 2550 5450 2550
-Wire Wire Line
-	6250 3300 6400 3300
-Wire Wire Line
-	6400 3300 6400 3100
-Connection ~ 6250 3300
-Wire Wire Line
-	6400 3100 6700 3100
-Connection ~ 6400 3100
-Connection ~ 6700 3100
-Wire Wire Line
-	6700 3100 7000 3100
-Wire Wire Line
-	6400 2900 6700 2900
-Connection ~ 6700 2900
-Wire Wire Line
-	6700 2900 7000 2900
-Text GLabel 7000 2900 1    50   Input ~ 0
-GND
-NoConn ~ 4650 3700
-NoConn ~ 6250 3900
-NoConn ~ 6250 3500
-Wire Wire Line
-	6250 3700 6700 3700
-Connection ~ 6700 3700
-Wire Wire Line
-	6700 3700 7000 3700
-Wire Wire Line
-	6700 3900 7000 3900
-Text GLabel 7000 3900 3    50   Input ~ 0
-GND
-Wire Wire Line
-	4650 3500 4400 3500
-Wire Wire Line
-	4400 3500 4400 3650
-Wire Wire Line
-	4400 3650 4350 3650
-Wire Wire Line
-	4150 3650 4150 3350
-Wire Wire Line
-	4150 3350 4100 3350
-Text GLabel 3700 3450 0    50   Input ~ 0
-CVBS
-Text GLabel 3700 3250 0    50   Input ~ 0
-LUMA
-$Comp
-L Device:R_Small_US R1
-U 1 1 5CF73400
-P 4550 3300
-F 0 "R1" H 4618 3346 50  0000 L CNN
-F 1 "470" H 4618 3255 50  0000 L CNN
-F 2 "Resistor_SMD:R_0603_1608Metric_Pad1.05x0.95mm_HandSolder" H 4550 3300 50  0001 C CNN
-F 3 "~" H 4550 3300 50  0001 C CNN
-	1    4550 3300
-	0    -1   -1   0
-$EndComp
-$Comp
-L Jumper:Jumper_3_Open JP1
-U 1 1 5CF744F6
-P 4400 2750
-F 0 "JP1" H 4400 2881 50  0000 C CNN
-F 1 "Jumper_3_Open" H 4400 2972 50  0000 C CNN
-F 2 "Connector_PinHeader_2.54mm:PinHeader_1x03_P2.54mm_Vertical" H 4400 2750 50  0001 C CNN
-F 3 "~" H 4400 2750 50  0001 C CNN
-	1    4400 2750
-	-1   0    0    1
-$EndComp
-Wire Wire Line
-	4650 3300 4650 2750
-Connection ~ 4650 3300
-Wire Wire Line
-	4450 3300 4150 3300
-Wire Wire Line
-	4150 3300 4150 2750
-Text GLabel 4400 2600 0    50   Input ~ 0
-CSYNC
-Text GLabel 5250 2550 0    50   Input ~ 0
-5V_IN
-Text GLabel 6500 4450 0    50   Input ~ 0
-CSYNC
-Text GLabel 6500 4350 0    50   Input ~ 0
-LUMA
-Text GLabel 6500 4550 0    50   Input ~ 0
-CVBS
-Text GLabel 6900 4450 2    50   Input ~ 0
-RCA_SYNC_OUT
-Text GLabel 6550 2550 0    50   Input ~ 0
-CSYNC
-Text GLabel 6550 2650 0    50   Input ~ 0
-CVBS
-Text GLabel 6550 2450 0    50   Input ~ 0
-LUMA
-Text GLabel 6950 2550 2    50   Input ~ 0
-VGA_SYNC_OUT
 Text GLabel 8250 2250 0    50   Input ~ 0
 RED_OUT
@@
 Text GLabel 8150 3950 0    50   Input ~ 0
 GND
+$Comp
+L Switch:SW_SPDT SW1
+U 1 1 5D1FECFC
+P 6150 2850
+F 0 "SW1" H 6150 2525 50  0000 C CNN
+F 1 "SW_SPDT" H 6150 2616 50  0000 C CNN
+F 2 "Tinkerplunk:C&K_SPDT" H 6150 2850 50  0001 C CNN
+F 3 "~" H 6150 2850 50  0001 C CNN
+	1    6150 2850
+	-1   0    0    1
+$EndComp
+Text GLabel 6350 2850 2    50   Input ~ 0
+VGA_SYNC_OUT
+Text GLabel 5950 2950 0    50   Input ~ 0
+CVBS
+Text GLabel 5950 2750 0    50   Input ~ 0
+LUMA
 $EndSCHEMATC
